File: hardware/pcb/luabot_v1/luabot_v1.kicad_pcb (KiCad board)
At the start: 2 copper layers, 0 parts

Commit message: avance hadware y librerias footprint
Parts:
- added C1, C2: 330µF, C1V7, F.Cu at (128.3, 108.0)
- added C3: 100pF, C1, F.Cu at (128.3, 108.0)
- added CON1: bat_in, BARREL_JACK, F.Cu at (36.8, 113.0)
- added JP1: jump_power_source, pin_socket_3, F.Cu at (128.3, 108.0)
- added JP2: JUMPER, pin_socket_2, F.Cu at (128.3, 108.0)
- added JP3: jump 3.3v or 5v, pin_socket_3, F.Cu at (128.3, 108.0)
- added P1: ext_izq_GPIO, pin_socket_9, F.Cu at (66.0, 54.6)
- added P2: ext_der_GPIO, pin_socket_9, F.Cu at (66.0, 77.5)
- added P3: uart, pin_socket_4, F.Cu at (128.3, 108.0)
- added P5: (GND,VCC)_GPIO, pin_socket_7x2, F.Cu at (44.5, 104.1)
- added P6: salidas_GPIO, pin_socket_7, F.Cu at (128.3, 108.0)
- added R1, R2, R3, R4, R5: 10k, R3, F.Cu at (128.3, 108.0)
- added R6: 100k, R3, F.Cu at (128.3, 108.0)
- added R7: 220k, R3, F.Cu at (128.3, 108.0)
- added SW1: SW_PUSH_SMALL, SW_PUSH_SMALL, F.Cu at (128.3, 108.0)
- added U1: ESP-07V2, ESP-07v2, F.Cu at (63.5, 66.0)
- added U2: LM1117-3.3V, SOT223, F.Cu at (128.3, 108.0)
Other:
- board outline added: 50.8 x 25.4 mm
