File: hardware/pcb/luabot_v1/luabot_v1.sch (KiCad schematic (older format))
At the start: 0 parts

Commit message: Creando primera versión de pcb luabot
Parts:
- added ASM1117_3.3V: CONN_3, symbol CONN_3
- added C1: 10pF, ~, symbol C
- added C2, C?: 330µF, ~, symbol CAPAPOL
- added CON1: BARREL_JACK, symbol BARREL_JACK
- added JP1, JP3: JUMPER3, ~, symbol JUMPER3
- added JP2: JUMPER, ~, symbol JUMPER
- added P1, P2: CONN_9, symbol CONN_9
- added P3: CONN_4, symbol CONN_4
- added P5: CONN_6X2, symbol CONN_6X2
- added P6: CONN_6, symbol CONN_6
- added R1, R2, R3, R4, R5: 10k, ~, symbol R
- added SW1: SW_PUSH_SMALL, ~, symbol SW_PUSH_SMALL
- added U1: ESP-07V2, symbol ESP-07V2
Connections:
- net labels added: +3.3V, +5V, +5V_CARGADOR, +5V_USB, 015, ADC, CH_PD, D0, D1, D2, D5, D6, D7, FLASH, GND, O02, O15, O2, RX, Reset, TX
- wire segments 0 -> 87

Commit message: agregando condicionamiento de condicionamiento digital
Parts:
- added 100k, 220k: R, ~, symbol R
Connections:
- net labels added: ADC_EX
- wire segments 87 -> 91

Commit message: avance hadware y librerias footprint
Parts:
- removed ASM1117_3.3V: CONN_3, symbol CONN_3
- removed P5: CONN_6X2, symbol CONN_6X2
- removed P6: CONN_6, symbol CONN_6
- added P5: (GND,VCC)_GPIO, symbol CONN_7X2
- added P6: salidas_GPIO, symbol CONN_7
- added U2: LM1117-3.3V, symbol LM1117-3.3V
- C3: renamed from C1; value 10pF -> 100pF
- CON1: value BARREL_JACK -> bat_in
- JP1: value JUMPER3 -> jump_power_source
- JP3: value JUMPER3 -> jump 3.3v or 5v
- P1: value CONN_9 -> ext_izq_GPIO
- P2: value CONN_9 -> ext_der_GPIO
- P3: value CONN_4 -> uart
- R6: renamed from 100k; value R -> 100k
- R7: renamed from 220k; value R -> 220k
- gave numbers to parts that had none: 1
Connections:
- net labels removed: 015, O2
- wire segments 91 -> 97
Other:
- moved on the sheet: C1, C2
