File: hardware/pcb/luabot_v2/luabot_v2.sch (KiCad schematic (older format))
At the start: 20 parts, among them CON1 bat_in, P3 uart, P5 (GND,VCC)_GPIO, P6 salidas_GPIO, SW1 SW_PUSH_SMALL, U1 ESP-07V2, U2 LM1117-3.3V

Commit message: avance hadware layout
Parts:
- removed P5: (GND,VCC)_GPIO, symbol CONN_7X2
- added P2: GND_GPIO, symbol CONN_7
- added P3: VCC_GPIO, symbol CONN_7
- renumbered P3 to P1, P6 to P4
Changed lines of the file:
@@
 $EndComp
 $Comp
-L CONN_4 P3
+L CONN_4 P1
 U 1 1 56AB909B
 P 1100 1550
-F 0 "P3" V 1050 1550 50  0000 C CNN
+F 0 "P1" V 1050 1550 50  0000 C CNN
 F 1 "uart" V 1150 1550 50  0000 C CNN
 F 2 "" H 1100 1550 60  0000 C CNN
@@
 L GND #PWR021
 U 1 1 56AB9CAF
-P 7150 3950
-F 0 "#PWR021" H 7150 3950 30  0001 C CNN
-F 1 "GND" H 7150 3880 30  0001 C CNN
-F 2 "" H 7150 3950 60  0000 C CNN
-F 3 "" H 7150 3950 60  0000 C CNN
-	1    7150 3950
+P 6700 3950
+F 0 "#PWR021" H 6700 3950 30  0001 C CNN
+F 1 "GND" H 6700 3880 30  0001 C CNN
+F 2 "" H 6700 3950 60  0000 C CNN
+F 3 "" H 6700 3950 60  0000 C CNN
+	1    6700 3950
 	1    0    0    -1
 $EndComp
@@
 $EndComp
 $Comp
-L CONN_7X2 P5
-U 1 1 56B2762B
-P 7550 3500
-F 0 "P5" H 7550 3900 60  0000 C CNN
-F 1 "(GND,VCC)_GPIO" V 7550 3500 60  0000 C CNN
-F 2 "" H 7550 3500 60  0000 C CNN
-F 3 "" H 7550 3500 60  0000 C CNN
-	1    7550 3500
-	1    0    0    -1
-$EndComp
-$Comp
-L CONN_7 P6
+L CONN_7 P4
 U 1 1 56B276B6
 P 9150 3600
-F 0 "P6" V 9120 3600 60  0000 C CNN
+F 0 "P4" V 9120 3600 60  0000 C CNN
 F 1 "salidas_GPIO" V 9220 3600 60  0000 C CNN
 F 2 "" H 9150 3600 60  0000 C CNN
@@
 	9650 1850 9550 1850
 Wire Wire Line
-	7150 3200 7150 3950
-Connection ~ 7150 3800
-Connection ~ 7150 3700
-Connection ~ 7150 3600
-Connection ~ 7150 3500
-Connection ~ 7150 3400
-Wire Wire Line
-	7950 2950 7950 3800
+	7700 2850 7600 2850
+Wire Wire Line
+	8300 2850 8200 2850
+Wire Wire Line
+	8800 3300 8650 3300
+Wire Wire Line
+	8300 3800 8800 3800
+Wire Wire Line
+	8800 3700 8650 3700
+Wire Wire Line
+	8800 3600 8450 3600
+Wire Wire Line
+	8800 3500 8650 3500
+Wire Wire Line
+	8800 3400 8450 3400
+Wire Wire Line
+	5700 4250 5700 4550
+Wire Wire Line
+	5150 4400 5700 4400
+Connection ~ 5700 4400
+Wire Wire Line
+	5700 3500 5700 3750
+Wire Wire Line
+	5700 5050 5700 5350
+Wire Wire Line
+	2450 2000 2450 1850
+Wire Wire Line
+	2450 1850 2800 1850
+Wire Wire Line
+	4200 1850 3850 1850
+Wire Wire Line
+	4000 2050 4000 2200
+Wire Wire Line
+	3850 2050 4000 2050
+Wire Wire Line
+	2600 2100 2600 2050
+Wire Wire Line
+	2600 2050 2800 2050
+Wire Wire Line
+	8700 3900 8800 3900
+Wire Wire Line
+	4200 1900 4200 1850
+$Comp
+L CONN_7 P2
+U 1 1 56B38504
+P 7050 3500
+F 0 "P2" V 7020 3500 60  0000 C CNN
+F 1 "GND_GPIO" V 7120 3500 60  0000 C CNN
+F 2 "" H 7050 3500 60  0000 C CNN
+F 3 "" H 7050 3500 60  0000 C CNN
+	1    7050 3500
+	1    0    0    -1
+$EndComp
+$Comp
+L CONN_7 P3
+U 1 1 56B38513
+P 7600 3500
+F 0 "P3" V 7570 3500 60  0000 C CNN
+F 1 "VCC_GPIO" V 7670 3500 60  0000 C CNN
+F 2 "" H 7600 3500 60  0000 C CNN
+F 3 "" H 7600 3500 60  0000 C CNN
+	1    7600 3500
+	-1   0    0    -1
+$EndComp
+Wire Wire Line
+	6700 3200 6700 3950
+Connection ~ 6700 3200
+Connection ~ 6700 3300
+Connection ~ 6700 3400
+Connection ~ 6700 3500
+Connection ~ 6700 3600
+Connection ~ 6700 3700
+Connection ~ 6700 3800
+Wire Wire Line
+	7950 3800 7950 2950
+Connection ~ 7950 3200
 Connection ~ 7950 3300
 Connection ~ 7950 3400
@@
 Connection ~ 7950 3600
 Connection ~ 7950 3700
-Wire Wire Line
-	7700 2850 7600 2850
-Wire Wire Line
-	8300 2850 8200 2850
-Wire Wire Line
-	8800 3300 8650 3300
-Wire Wire Line
-	8300 3800 8800 3800
-Wire Wire Line
-	8800 3700 8650 3700
-Wire Wire Line
-	8800 3600 8450 3600
-Wire Wire Line
-	8800 3500 8650 3500
-Wire Wire Line
-	8800 3400 8450 3400
-Wire Notes Line
-	7000 2650 7000 4050
-Wire Notes Line
-	7000 4050 9350 4050
-Wire Notes Line
-	9350 4050 9350 2650
-Wire Notes Line
-	9350 2650 7000 2650
-Wire Wire Line
-	5700 4250 5700 4550
-Wire Wire Line
-	5150 4400 5700 4400
-Connection ~ 5700 4400
-Wire Wire Line
-	5700 3500 5700 3750
-Wire Wire Line
-	5700 5050 5700 5350
-Wire Wire Line
-	2450 2000 2450 1850
-Wire Wire Line
-	2450 1850 2800 1850
-Wire Wire Line
-	4200 1850 3850 1850
-Wire Wire Line
-	4000 2050 4000 2200
-Wire Wire Line
-	3850 2050 4000 2050
-Wire Wire Line
-	2600 2100 2600 2050
-Wire Wire Line
-	2600 2050 2800 2050
-Connection ~ 7150 3300
-Connection ~ 7950 3200
-Connection ~ 7150 3200
 Connection ~ 7950 3800
-Wire Wire Line
-	8700 3900 8800 3900
-Wire Wire Line
-	4200 1900 4200 1850
 $EndSCHEMATC
