File: hardware/pcb/switchPower/switchPower.sch (KiCad schematic (older format))
At the start: 0 parts

Commit message: avance switchporwer esquematico
Parts:
- added 1N4004: DIODE, ~, symbol DIODE
- added K0: CONN_3, symbol CONN_3
- added K1: RELAY_5V, ~, symbol RELAY_5V
- added NPN1: 2N2222, ~, symbol NPN
- added NPN2: 2N2222A, ~, symbol NPN
- added P2, P3, P4: CONN_2, symbol CONN_2
- added R1: 10K, ~, symbol R
- added R2: 30k, ~, symbol R
Connections:
- net labels added: GND, IN, VCC
- wire segments 0 -> 29
- no-connect marks 0 -> 1

Commit message: avance switchpower
Parts:
- removed K1: RELAY_5V, ~, symbol RELAY_5V
- added RLY5: RELAY_5PINS, symbol RELAY_5PINS
Connections:
- wire segments 29 -> 27
Changed lines of the file:
@@
 LIBS:contrib
 LIBS:valves
+LIBS:w_relay
 LIBS:switchPower-cache
 EELAYER 27 0
@@
 $EndComp
 $Comp
-L RELAY_5V K1
-U 1 1 56B55B37
-P 3450 1150
-F 0 "K1" H 3400 1550 70  0000 C CNN
-F 1 "RELAY_5V" H 3600 650 70  0000 C CNN
-F 2 "~" H 3450 1150 60  0000 C CNN
-F 3 "~" H 3450 1150 60  0000 C CNN
-	1    3450 1150
-	1    0    0    -1
-$EndComp
-$Comp
 L CONN_2 P3
 U 1 1 56B55B87
@@
 	0    1    1    0
 $EndComp
-NoConn ~ 3850 1100
 $Comp
 L NPN NPN1
@@
 	1600 850  1600 750
 Wire Wire Line
-	2450 850  2900 850
-Wire Wire Line
 	2450 850  2450 1100
 Connection ~ 2700 850
 Wire Wire Line
-	2450 1500 3050 1500
-Wire Wire Line
 	2700 850  2700 650
 Wire Wire Line
-	2900 850  2900 1400
-Wire Wire Line
-	2900 1400 3050 1400
-Wire Wire Line
 	4450 1100 4400 1100
 Wire Wire Line
 	4400 1100 4400 1500
 Wire Wire Line
-	3850 1300 4200 1300
-Wire Wire Line
-	4200 1300 4200 1500
-Wire Wire Line
-	3950 1200 4200 1200
-Wire Wire Line
-	4200 1200 4200 900
-Wire Wire Line
-	4200 900  4450 900
+	2700 2200 2700 2400
+Wire Wire Line
+	2250 2000 2400 2000
+Wire Wire Line
+	1600 2000 1750 2000
+Wire Wire Line
+	6200 1400 6350 1400
+Wire Wire Line
+	5550 1400 5700 1400
+Wire Wire Line
+	6650 1200 6650 1100
+Wire Wire Line
+	6650 1100 6850 1100
+Wire Wire Line
+	6850 900  6650 900
+Wire Wire Line
+	6650 900  6650 850
+Wire Wire Line
+	6650 1600 6650 1900
+Wire Wire Line
+	2700 1800 2700 1500
+Wire Wire Line
+	2450 850  3350 850
+Wire Wire Line
+	3350 850  3350 1100
+$Comp
+L RELAY_5PINS RLY5
+U 1 1 56B6242E
+P 3750 1300
+F 0 "RLY5" H 3750 1550 60  0000 C CNN
+F 1 "RELAY_5PINS" H 3750 1150 60  0000 C CNN
+F 2 "" H 3750 1300 60  0000 C CNN
+F 3 "" H 3750 1300 60  0000 C CNN
+	1    3750 1300
+	0    -1   -1   0
+$EndComp
+Wire Wire Line
+	2450 1500 3600 1500
 Connection ~ 2700 1500
 Wire Wire Line
-	2700 2200 2700 2400
-Wire Wire Line
-	2250 2000 2400 2000
-Wire Wire Line
-	1600 2000 1750 2000
-Wire Wire Line
-	6200 1400 6350 1400
-Wire Wire Line
-	5550 1400 5700 1400
-Wire Wire Line
-	6650 1200 6650 1100
-Wire Wire Line
-	6650 1100 6850 1100
-Wire Wire Line
-	6850 900  6650 900
-Wire Wire Line
-	6650 900  6650 850
-Wire Wire Line
-	6650 1600 6650 1900
-Wire Wire Line
-	2700 1800 2700 1500
+	3350 1100 3600 1100
+NoConn ~ 3850 1100
+Wire Wire Line
+	3750 1100 3750 900
+Wire Wire Line
+	3750 900  4450 900
+Wire Wire Line
+	3800 1500 4200 1500
 $EndSCHEMATC
