File: hardware/pcb/switchPower/switchPower.kicad_pcb (KiCad board)
At the start: 2 copper layers, 42.1 x 34.9 mm, 11 parts, among them K0 CONN_3, P2 CON_120V_IN, P3 CON_120V_OUT, P4 CONN_2

Commit message: Costos trajeta y kit
Routing:
- net N-0000011: track 56.4 -> 50.9 mm
- removed copper zone on B.Cu, net GND
Changed lines of the file:
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@@
     (links 15)
     (no_connects 0)
-    (area 113.424999 25.524999 175.077382 74.489756)
+    (area 113.4 25.524999 178.633251 75.802295)
     (thickness 1.6)
     (drawings 9)
@@
   (segment (start 151.3 54.78) (end 140.32 54.78) (width 3) (layer B.Cu) (net 4))
   (segment (start 140.32 54.78) (end 139.1 56) (width 3) (layer B.Cu) (net 4))
-  (segment (start 120.8 56) (end 120.8 49.5) (width 1) (layer B.Cu) (net 5))
-  (segment (start 140.87 34.47) (end 139.87 34.47) (width 1) (layer B.Cu) (net 5))
-  (segment (start 143.7 37.3) (end 140.87 34.47) (width 1) (layer B.Cu) (net 5))
-  (segment (start 143.7 47.4) (end 143.7 37.3) (width 1) (layer B.Cu) (net 5))
-  (segment (start 137.8 47.4) (end 143.7 47.4) (width 1) (layer B.Cu) (net 5))
-  (segment (start 136.9 46.5) (end 137.8 47.4) (width 1) (layer B.Cu) (net 5))
-  (segment (start 123.8 46.5) (end 136.9 46.5) (width 1) (layer B.Cu) (net 5))
-  (segment (start 120.8 49.5) (end 123.8 46.5) (width 1) (layer B.Cu) (net 5))
+  (segment (start 120.8 56) (end 120.8 49) (width 1.3) (layer B.Cu) (net 5))
+  (segment (start 143.5 38.1) (end 139.87 34.47) (width 1.3) (layer B.Cu) (net 5))
+  (segment (start 143.5 40.3) (end 143.5 38.1) (width 1.3) (layer B.Cu) (net 5))
+  (segment (start 142.3 41.5) (end 143.5 40.3) (width 1.3) (layer B.Cu) (net 5))
+  (segment (start 135.7 41.5) (end 142.3 41.5) (width 1.3) (layer B.Cu) (net 5))
+  (segment (start 130.6 46.6) (end 135.7 41.5) (width 1.3) (layer B.Cu) (net 5))
+  (segment (start 123.2 46.6) (end 130.6 46.6) (width 1.3) (layer B.Cu) (net 5))
+  (segment (start 120.8 49) (end 123.2 46.6) (width 1.3) (layer B.Cu) (net 5))
   (segment (start 118.4 57.81) (end 118.4 56) (width 1) (layer B.Cu) (net 5))
   (segment (start 118.4 56) (end 120.8 56) (width 1) (layer B.Cu) (net 5))
@@
   (segment (start 127.7 43.2) (end 126.9 44) (width 1) (layer B.Cu) (net 10))
   (segment (start 118.4 50.19) (end 118.4 46.27) (width 1.3) (layer B.Cu) (net 10))
-  (zone (net 1) (net_name GND) (layer B.Cu) (hatch edge 0.508)
-    (connect_pads (clearance 0.508))
-    (min_thickness 0.4)
-    (fill (arc_segments 16) (thermal_gap 0.508) (thermal_bridge_width 0.508))
-    (polygon
-      (pts
-        (xy 131.3 26.9) (xy 137.8 26.9) (xy 146.3 26.9) (xy 151.8 32.4) (xy 154.1 32.4)
-        (xy 154 58.8) (xy 137.4 58.8) (xy 134.1 55.5) (xy 130.6 55.5) (xy 127.1 59)
-        (xy 120.2 59) (xy 119.6 59.4) (xy 116.6 59.4) (xy 116.6 30.8) (xy 120.5 26.9)
-      )
-    )
-  )
 )

Commit message: Costos y modificaciones menores para finaluzar producto
Parts:
- moved G*** 8.05 mm to (150.9, 29.2)
Routing:
- net N-0000011: track 50.9 -> 70.4 mm
- net GND: track 27.5 -> 26.0 mm
- added copper zone on B.Cu, net GND
Other:
- outline, holes or cut-outs redrawn
