File: hardware/pcb/cp_luabot_v2/luabot_v2.kicad_pcb (KiCad board)
At the start: 2 copper layers, 67.8 x 32.1 mm, 26 parts, among them CON1 BAT_IN, P2 GND_GPIO, P3 VCC_GPIO, SW1 RESET, U1 ESP-07V2, U2 LM1117

Commit message: arreglando hardware, finalizando muestras
Parts:
- removed the G*** at (21.1, 41.1)
- removed the G*** at (84.3, 27.2)
- moved G*** 0.13 mm to (21.5, 47.6)
Other:
- board text added: "3.3V"
- board text added: "5V_BAT_IN"
- board text added: "VCC"
- board text removed: "3.3V ←"
- board text removed: "5VBAT_IN"
- board text removed: "https://bitbucket.org/pinguinotux/luabot"
- board text removed: "↑ VCC"
- board text removed: "↓VCC"
